File: boards/reference-esp32s3/sensor-subcircuit.kicad_sch (KiCad schematic)
At the start: 4 parts, among them U2 BME280

Commit message: Passives resolve to registry ids; ADR-0004 amends ADR-0003's authoring concession
R1/R2/C1 now carry opc_id (electronic/r-0603, electronic/c-0603), so every schematic BOM line resolves to a cited entry. ERC still 0 violations. ADR-0004 records that ADR-0003 overstated the loss from dropping atopile: the netlist description is the source and the .kicad_sch is a build artifact, so diffable reviewable circuit source survived. What is genuinely still worse is named: no type system over connections, no module package manager, no layout aesthetics.
Parts:
- C1: opc_id (none) -> electronic/c-0603
- R1, R2: opc_id (none) -> electronic/r-0603
Changed lines of the file:
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@@
 				"sensor-subcircuit"
 				(path
-					"/b600e005-c347-4ca8-9e61-727d6a834484"
+					"/c85bf385-429b-4258-8358-4918491b061c"
 					(reference "U2")
 					(unit 1)
@@
 			)
 		)
-		(instances
-			(project
-				"sensor-subcircuit"
-				(path
-					"/b600e005-c347-4ca8-9e61-727d6a834484"
+		(property
+			"opc_id"
+			"electronic/r-0603"
+			(at 140.0 100.0 0)
+			(effects
+				(font
+					(size 1.27 1.27)
+				)
+				(hide yes)
+			)
+		)
+		(instances
+			(project
+				"sensor-subcircuit"
+				(path
+					"/c85bf385-429b-4258-8358-4918491b061c"
 					(reference "R1")
 					(unit 1)
@@
 			)
 		)
-		(instances
-			(project
-				"sensor-subcircuit"
-				(path
-					"/b600e005-c347-4ca8-9e61-727d6a834484"
+		(property
+			"opc_id"
+			"electronic/r-0603"
+			(at 150.0 100.0 0)
+			(effects
+				(font
+					(size 1.27 1.27)
+				)
+				(hide yes)
+			)
+		)
+		(instances
+			(project
+				"sensor-subcircuit"
+				(path
+					"/c85bf385-429b-4258-8358-4918491b061c"
 					(reference "R2")
 					(unit 1)
@@
 			)
 		)
-		(instances
-			(project
-				"sensor-subcircuit"
-				(path
-					"/b600e005-c347-4ca8-9e61-727d6a834484"
+		(property
+			"opc_id"
+			"electronic/c-0603"
+			(at 160.0 100.0 0)
+			(effects
+				(font
+					(size 1.27 1.27)
+				)
+				(hide yes)
+			)
+		)
+		(instances
+			(project
+				"sensor-subcircuit"
+				(path
+					"/c85bf385-429b-4258-8358-4918491b061c"
 					(reference "C1")
 					(unit 1)
@@
 				"sensor-subcircuit"
 				(path
-					"/b600e005-c347-4ca8-9e61-727d6a834484"
+					"/c85bf385-429b-4258-8358-4918491b061c"
 					(reference "#FLG01")
 					(unit 1)
@@
 				"sensor-subcircuit"
 				(path
-					"/b600e005-c347-4ca8-9e61-727d6a834484"
+					"/c85bf385-429b-4258-8358-4918491b061c"
 					(reference "#FLG02")
 					(unit 1)
